Commit message: updated multi object for point following

File: resources/objects/urdf_models/models/green_cup/model.urdf (robot description, URDF)
Before this commit: robot model.urdf, 1 links, 0 joints
Links:
- link baseLink: geometry collision mesh filename=collision.obj scale=3 3 3; visual mesh filename=textured.obj scale=3 3 3

File: resources/objects/urdf_models/models/knife/model.urdf (robot description, URDF)
Before this commit: robot model.urdf, 1 links, 0 joints
Links:
- link baseLink: geometry collision mesh filename=collision.obj scale=3 3 3; visual mesh filename=textured.obj scale=3 3 3

File: resources/objects/urdf_models/models/orion_pie/model.urdf (robot description, URDF)
Before this commit: robot model.urdf, 1 links, 0 joints
Links:
- link baseLink: geometry collision mesh filename=collision.obj scale=3 3 3; visual mesh filename=textured.obj scale=3 3 3
